File: hardware/pcb/detergent-dispenser.kicad_pcb (KiCad board)
At the start: 2 copper layers, 53.3 x 43.2 mm, 12 parts, among them J1 RJ45 (Bartendro), J2 User Button, J3 20v Input, SW1 Reset, U1 MIC2940A-5.0WU

Commit message: Add a note to PCB about 5v protection
Other:
- board text added: "Notes: - The 5v going to the TinyPICO should be protected byt a diode or something to prevent conflics when USB is connected"
